File: hardware/eagle/tinySensor.sch (EAGLE design)
At the start: 0 parts

Commit message: Schematics redrawn, work in progress
Parts:
- added C1: 100nF, 0SBLib:C0805
- added C2: 10uF, 0SBLib:C0805
- added C3: 1uF, rcl:CPOL-EUC
- added J1, J5, J7: (no value), 0SBLib:M03PTH
- added J3: (no value), SparkFun-Connectors:M06SIP
- added J6: (no value), SparkFun-Connectors:M03X2SHROUD
- added JP1: (no value), SparkFun-Retired:JUMPER-2PTH
- added LED: (no value), 0SBLib:LED3MM
- added R1: 1k, 0SBLib:R0805
- added R2, R3, R6: 4.7k, 0SBLib:R0805
- added R4: 75, 0SBLib:R0805
- added U$1: ATTINY84ATTINY84-20PU, SparkFun-DigitalIC:ATTINY84ATTINY84-20PU
Connections:
- new net ANALOG_SENSOR: J7.2, R4.2, U$1.(PCINT0/AREF/ADC0)PA0
- new net AUX: U$1.(PCINT10/INT0/OC0A/CKOUT)PB2
- new net BATTERY_CHECKER: U$1.(PCINT1/AIN0/ADC1)PA1
- new net GND: C1.1, C2.1, C3.-, J1.1, J3.2, J3.6, J5.2, J6.6, J7.1, LED.C, U$1.GND
- new net LED_OUT: JP1.1, U$1.(PCINT9/XTAL2)PB1
- new net MISO: J6.1, U$1.(PCINT5/OC1B/MISO/DO/ADC5)PA5
- new net N$1: JP1.2, R1.1
- new net N$2: LED.A, R1.2
- new net N$4: C3.+, R4.1
- new net ONEWIRE: J5.1, R6.1, U$1.(PCINT3/T0/ADC3)PA3
- new net PWM_OUT: U$1.(PCINT7/ICP/OC0B/ADC7)PA7
- new net RESET: J6.5, U$1.(PCINT11/~RESET/DW)PB3
- new net SCL/SCK: J6.3, U$1.(PCINT4/T1/SCL/USCK/ADC4)PA4
- new net SCL_SCK: J3.3, R3.1
- new net SDA/MOSI: J3.4, J6.4, R2.1, U$1.(PCINT6/OC1A/SDA/MOSI/ADC6)PA6
- new net SENSOR_VCC: J3.1, J5.3, J7.3, R2.2, R3.2, R6.2, U$1.(PCINT2/AIN1/ADC2)PA2
- new net TX_RADIO: J1.3, U$1.(PCINT8/XTAL1/CLKI)PB0
- new net VCC: C1.2, C2.2, J1.2, J6.2, U$1.VCC
Other:
- note added: "Analog Sensor"
- note added: "BMP/BME Breakout"
- note added: "OneWire Sensor"
- note added: "Optional filter for LM35 sensor"
